Commit message: ..

File: Machines/test 3/test3.urdf (robot description, URDF)
Before this commit: robot test-bot, 1 links, 0 joints
Links:
- removed link boat
- added link base_frame, mass 0.0; collision box size=0.0 0.0 0.0; visual box size=0.0 0.0 0.0
- added link boat_joint, mass 27.0; collision mesh filename=stl/Part Studio - båt.stl scale=1.0; visual mesh filename=stl/Part Studio - båt.stl scale=1.0
- added link world

Commit message: ..

File: Machines/test 3/test3.urdf (robot description, URDF)
Before this commit: robot test-bot, 3 links, 0 joints
Links:
- link base_frame: geometry collision box size=1.0 1.0 1.0; visual box size=1.0 1.0 1.0
- link boat_joint: geometry collision box size=1.0 1.0 1.0; visual box size=1.0 1.0 1.0

Commit message: .

File: Machines/test 3/test3.urdf (robot description, URDF)
Before this commit: robot test-bot, 3 links, 0 joints
Links:
- removed link base_frame
- removed link boat_joint
- removed link world
- added link boat_link, mass 0.0; collision box size=1.0 1.0 1.0; visual box size=0.0 0.0 0.0
- added link map
Joints:
- added joint boat_joint: type revolute, parent map, child boat_link, origin xyz=0 0 0 rpy=0 0 0, axis 0 0 0, limit lower=-3.14159 upper=3.14159 effort=1000.0 velocity=50.0
